File: IOTide-0x40/IOTide-0x40.kicad_pcb (KiCad board)
At the start: 2 copper layers, 166 x 61 mm, 239 parts, among them J1 NEO, J10 Conn_01x05, J11 V+, J12 DAISY, J13 Conn_01x05, J14 Conn_01x05, J15 Conn_01x05, J16 Conn_01x05, J17 Conn_01x05, J18 Conn_01x05, J19 Conn_01x05, J2 KH-TYPE-C-16P, J20 Conn_01x05, J21 DAISY, J3 S1, J4 S2, J5 Conn_01x05, J6 Conn_01x05, J7 Conn_01x05, J8 Conn_01x05, J9 Conn_01x05, SW1 RST, SW2 ADDR, SW3 BOOT, U1 STM32F407VETx, U10 ULN2803A, U11 ULN2803A, U12 ULN2803A, U13 ULN2803A, U14 ULN2803A, U2 AMS1117-3.3, U3 USBLC6-2SC6, U4 D5V0P4UR6SO, U5 D5V0P4UR6SO, U6 D5V0P4UR6SO, U7 ULN2803A, U8 ULN2803A, U9 ULN2803A

Commit message: wip
Parts:
- added J23: GPIO, Connector_PinHeader_2.54mm:PinHeader_1x12_P2.54mm_Vertical, F.Cu at (121.0, 71.0)
- added U15: DRV8833PWP, Package_SO:HTSSOP-16-1EP_4.4x5mm_P0.65mm_EP3.4x5mm_Mask2.46x2.31mm_ThermalVias, F.Cu at (301.1, 38.4)
- added U16: DRV8833RTY, Package_DFN_QFN:Texas_RTY_WQFN-16-1EP_4x4mm_P0.65mm_EP2.1x2.1mm_ThermalVias, F.Cu at (307.5, 50.6)
- moved R67 206.1 mm to (259.5, 19.5), turned to -90 degrees
- moved R66 202.5 mm to (256.5, 19.5), turned to -90 degrees
- moved R71 202.5 mm to (259.5, 38.0), turned to -90 degrees
- moved R65 199.0 mm to (253.5, 19.5), turned to -90 degrees
- moved R70 199.0 mm to (256.5, 38.0), turned to -90 degrees
- moved R59 196.7 mm to (243.0, 19.5), turned to -90 degrees
- moved R64 195.5 mm to (250.5, 19.5), turned to -90 degrees
- moved R69 195.5 mm to (253.5, 38.0), turned to -90 degrees
- moved R58 193.1 mm to (240.0, 19.5), turned to -90 degrees
- moved R68 192.0 mm to (250.5, 38.0), turned to -90 degrees
- moved D61 191.6 mm to (255.0, 19.5), turned to 90 degrees
- moved R57 189.6 mm to (237.0, 19.5), turned to -90 degrees
- moved R72 189.5 mm to (254.5, 73.2), turned to 180 degrees
- moved D60 188.0 mm to (252.0, 19.5), turned to 90 degrees
- moved R4 186.6 mm to (239.0, 72.3)
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- renumbered SW2 to ADDR1, SW3 to BOOT0, SW1 to RST1
Connections:
- D10 pad 2: /S2P4 -> S2P4
- D11 pad 2: /S3P1 -> S3P1
- D12 pad 2: /S3P2 -> S3P2
- D13 pad 2: /S3P3 -> S3P3
- D14 pad 2: /S3P4 -> S3P4
- D15 pad 2: /S4P1 -> S4P1
- D16 pad 2: /S4P2 -> S4P2
- D17 pad 2: /S4P3 -> S4P3
- D18 pad 2: /S4P4 -> S4P4
- D23 pad 2: /S6P1 -> S6P1
- D24 pad 2: /S6P2 -> S6P2
- D25 pad 2: /S6P3 -> S6P3
- D26 pad 2: /S6P4 -> S6P4
- D27 pad 2: /S7P1 -> S7P1
- D28 pad 2: /S7P2 -> S7P2
- D29 pad 2: /S7P3 -> S7P3
- D30 pad 2: /S7P4 -> S7P4
- D31 pad 2: /S8P1 -> S8P1
- D32 pad 2: /S8P2 -> S8P2
- D33 pad 2: /S8P3 -> S8P3
- D34 pad 2: /S8P4 -> S8P4
- D7 pad 2: /S2P1 -> S2P1
- D8 pad 2: /S2P2 -> S2P2
- D9 pad 2: /S2P3 -> S2P3
- U1 pad 1: S1P2 -> /S16P2
- U1 pad 15: S1P1 -> /S14P4
- U1 pad 16: S1P2 -> /S14P3
- U1 pad 17: S1P3 -> /S14P2
- U1 pad 18: S1P4 -> /S14P1
- U1 pad 2: S1P1 -> /S16P1
- U1 pad 3: S1P4 -> /S15P4
- U1 pad 33: S1P1 -> S6P1
- U1 pad 34: S1P2 -> S6P2
- U1 pad 37: S1P1 -> S2P1
- U1 pad 38: S1P1 -> /S15P1
- U1 pad 39: S1P4 -> /S12P4
- U1 pad 4: S1P3 -> /S15P3
- U1 pad 40: S1P3 -> /S12P3
- U1 pad 41: S1P2 -> /S12P2
- U1 pad 42: S1P1 -> /S12P1
- U1 pad 43: S1P4 -> /S11P4
- U1 pad 44: S1P3 -> /S11P3
- U1 pad 45: S1P2 -> /S11P2
- U1 pad 46: S1P1 -> /S11P1
- U1 pad 47: S1P3 -> S3P3
- U1 pad 48: S1P4 -> S3P4
- U1 pad 5: S1P2 -> /S15P2
- U1 pad 51: S1P1 -> S4P1
- U1 pad 52: S1P2 -> S4P2
- U1 pad 53: S1P3 -> S4P3
- U1 pad 54: S1P4 -> S4P4
- U1 pad 55: S1P4 -> /S9P1
- U1 pad 56: S1P3 -> /S9P2
- U1 pad 57: S1P2 -> /S9P3
- U1 pad 58: S1P1 -> /S9P4
- U1 pad 59: S1P4 -> /S10P1
- U1 pad 60: S1P3 -> /S10P2
- U1 pad 61: S1P2 -> /S10P3
- U1 pad 62: S1P1 -> /S10P4
- U1 pad 63: S1P3 -> S6P3
- U1 pad 64: S1P4 -> S6P4
- U1 pad 65: S1P1 -> S7P1
- U1 pad 66: S1P2 -> S7P2
- U1 pad 7: S1P2 -> S8P2
- U1 pad 78: S1P3 -> S7P3
- U1 pad 79: S1P4 -> S7P4
- U1 pad 8: S1P3 -> S8P3
- U1 pad 80: S1P1 -> S8P1
- U1 pad 81: S1P4 -> /S13P1
- U1 pad 82: S1P3 -> /S13P2
- U1 pad 83: S1P2 -> /S13P3
- U1 pad 84: S1P1 -> /S13P4
- U1 pad 85: S1P4 -> /S5P1
- U1 pad 86: S1P3 -> /S5P2
- U1 pad 87: S1P2 -> /S5P3
- U1 pad 88: S1P1 -> /S5P4
- U1 pad 89: S1P2 -> S2P2
- U1 pad 9: S1P4 -> S8P4
- U1 pad 90: S1P3 -> S2P3
- U1 pad 91: S1P4 -> S2P4
- U1 pad 95: S1P1 -> S3P1
- U1 pad 96: S1P2 -> S3P2
- U1 pad 97: S1P4 -> /S16P4
- U1 pad 98: S1P3 -> /S16P3
- U10 pad 1: /S7P1 -> S7P1
- U10 pad 2: /S7P2 -> S7P2
- U10 pad 3: /S7P3 -> S7P3
- U10 pad 4: /S7P4 -> S7P4
- U10 pad 5: /S8P1 -> S8P1
- U10 pad 6: /S8P2 -> S8P2
- U10 pad 7: /S8P3 -> S8P3
- U10 pad 8: /S8P4 -> S8P4
- U7 pad 5: /S2P1 -> S2P1
- U7 pad 6: /S2P2 -> S2P2
- U7 pad 7: /S2P3 -> S2P3
- U7 pad 8: /S2P4 -> S2P4
- U8 pad 1: /S3P1 -> S3P1
- U8 pad 2: /S3P2 -> S3P2
- U8 pad 3: /S3P3 -> S3P3
- U8 pad 4: /S3P4 -> S3P4
- U8 pad 5: /S4P1 -> S4P1
- U8 pad 6: /S4P2 -> S4P2
- U8 pad 7: /S4P3 -> S4P3
- U8 pad 8: /S4P4 -> S4P4
- U9 pad 5: /S6P1 -> S6P1
- U9 pad 6: /S6P2 -> S6P2
- U9 pad 7: /S6P3 -> S6P3
- U9 pad 8: /S6P4 -> S6P4
Routing:
- net S1P4: track 0.00 -> 44.9 mm
- net S1P3: track 0.00 -> 41.5 mm
- net S1P2: track 0.00 -> 38.5 mm
- net S1P1: track 0.00 -> 35.1 mm
- net Net-(J3-Pin_4): track 0.00 -> 28.5 mm, vias 0 -> 1
- net +V: track 0.00 -> 28.1 mm
- net Net-(J3-Pin_3): track 0.00 -> 26.7 mm, vias 0 -> 1
- net Net-(J3-Pin_2): track 0.00 -> 24.9 mm, vias 0 -> 1
- net Net-(J3-Pin_1): track 0.00 -> 23.9 mm, vias 0 -> 1
- net Net-(J17-Pin_5): track 0.00 -> 21.1 mm
- net Net-(J15-Pin_5): track 0.00 -> 21.0 mm
- net Net-(J13-Pin_5): track 0.00 -> 20.9 mm
- net Net-(J19-Pin_5): track 0.00 -> 20.9 mm
- net Net-(J5-Pin_5): track 0.00 -> 20.6 mm
- net Net-(J7-Pin_5): track 0.00 -> 20.6 mm
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Other:
- copper layers 2 -> 4
