File: IOTide-0x40/IOTide-0x40.kicad_sch (KiCad schematic)
At the start: 239 parts, among them J1 NEO, J10 Conn_01x05, J11 V+, J12 DAISY, J13 Conn_01x05, J14 Conn_01x05, J15 Conn_01x05, J16 Conn_01x05, J17 Conn_01x05, J18 Conn_01x05, J19 Conn_01x05, J2 KH-TYPE-C-16P, J20 Conn_01x05, J21 DAISY, J3 S1, J4 S2, J5 Conn_01x05, J6 Conn_01x05, J7 Conn_01x05, J8 Conn_01x05, J9 Conn_01x05, SW1 RST, SW2 ADDR, SW3 BOOT, U1 STM32F407VETx, U10 ULN2803A, U11 ULN2803A, U12 ULN2803A, U13 ULN2803A, U14 ULN2803A, U2 AMS1117-3.3, U3 USBLC6-2SC6, U4 D5V0P4UR6SO, U5 D5V0P4UR6SO, U6 D5V0P4UR6SO, U7 ULN2803A, U8 ULN2803A, U9 ULN2803A

Commit message: wip
Parts:
- added J23: GPIO, Connector_PinHeader_2.54mm:PinHeader_1x12_P2.54mm_Vertical, symbol Connector_Generic:Conn_01x12
- added U15: DRV8833PWP, Package_SO:HTSSOP-16-1EP_4.4x5mm_P0.65mm_EP3.4x5mm_Mask2.46x2.31mm_ThermalVias, symbol Driver_Motor:DRV8833PWP
- renumbered SW2 to ADDR1, SW3 to BOOT0, SW1 to RST1
Connections:
- net +3V3: now also J23.4 (Pin_4)
- net GND: now also J23.3 (Pin_3)
- net MISO: now also J23.10 (Pin_10)
- net MOSI: now also J23.11 (Pin_11)
- net PB0: now also J23.5 (Pin_5)
- net PB1: now also J23.6 (Pin_6)
- net PH1: now also J23.12 (Pin_12)
- net RX: now also J23.2 (Pin_2)
- net S10P1: now also U1.59 (PD12)
- net S10P2: now also U1.60 (PD13)
- net S10P3: now also U1.61 (PD14)
- net S10P4: now also U1.62 (PD15)
- net S11P1: now also U1.46 (PE15)
- net S11P2: now also U1.45 (PE14)
- net S11P3: now also U1.44 (PE13)
- net S11P4: now also U1.43 (PE12)
- net S12P1: now also U1.42 (PE11)
- net S12P2: now also U1.41 (PE10)
- net S12P3: now also U1.40 (PE9)
- net S12P4: now also U1.39 (PE8)
- net S13P1: now also U1.81 (PD0)
- net S13P2: now also U1.82 (PD1)
- net S13P3: now also U1.83 (PD2)
- net S13P4: now also U1.84 (PD3)
- net S14P1: now also U1.18 (PC3)
- net S14P2: now also U1.17 (PC2)
- net S14P3: now also U1.16 (PC1)
- net S14P4: now also U1.15 (PC0)
- net S15P1: now also U1.38 (PE7)
- net S15P2: now also U1.5 (PE6)
- net S15P3: now also U1.4 (PE5)
- net S15P4: now also U1.3 (PE4)
- net S16P1: now also U1.2 (PE3)
- net S16P2: now also U1.1 (PE2)
- net S16P3: now also U1.98 (PE1)
- net S16P4: now also U1.97 (PE0)
- net S1P1: no longer U1.15 (PC0), U1.2 (PE3), U1.33 (PC4), U1.37 (PB2), U1.38 (PE7), U1.42 (PE11), U1.46 (PE15), U1.51 (PB12), U1.58 (PD11), U1.62 (PD15), U1.65 (PC8), U1.80 (PC12), U1.84 (PD3), U1.88 (PD7), U1.95 (PB8)
- net S1P2: no longer U1.1 (PE2), U1.16 (PC1), U1.34 (PC5), U1.41 (PE10), U1.45 (PE14), U1.5 (PE6), U1.52 (PB13), U1.57 (PD10), U1.61 (PD14), U1.66 (PC9), U1.7 (PC13), U1.83 (PD2), U1.87 (PD6), U1.89 (PB3), U1.96 (PB9)
- net S1P3: no longer U1.17 (PC2), U1.4 (PE5), U1.40 (PE9), U1.44 (PE13), U1.47 (PB10), U1.53 (PB14), U1.56 (PD9), U1.60 (PD13), U1.63 (PC6), U1.78 (PC10), U1.8 (PC14), U1.82 (PD1), U1.86 (PD5), U1.90 (PB4), U1.98 (PE1)
- net S1P4: no longer U1.18 (PC3), U1.3 (PE4), U1.39 (PE8), U1.43 (PE12), U1.48 (PB11), U1.54 (PB15), U1.55 (PD8), U1.59 (PD12), U1.64 (PC7), U1.79 (PC11), U1.81 (PD0), U1.85 (PD4), U1.9 (PC15), U1.91 (PB5), U1.97 (PE0)
- net S2P1: now also U1.37 (PB2)
- net S2P2: now also U1.89 (PB3)
- net S2P3: now also U1.90 (PB4)
- net S2P4: now also U1.91 (PB5)
- net S3P1: now also U1.95 (PB8)
- net S3P2: now also U1.96 (PB9)
- net S3P3: now also U1.47 (PB10)
- net S3P4: now also U1.48 (PB11)
- net S4P1: now also U1.51 (PB12)
- net S4P2: now also U1.52 (PB13)
- net S4P3: now also U1.53 (PB14)
- net S4P4: now also U1.54 (PB15)
- net S5P1: now also U1.85 (PD4)
- net S5P2: now also U1.86 (PD5)
- net S5P3: now also U1.87 (PD6)
- net S5P4: now also U1.88 (PD7)
- net S6P1: now also U1.33 (PC4)
- net S6P2: now also U1.34 (PC5)
- net S6P3: now also U1.63 (PC6)
- net S6P4: now also U1.64 (PC7)
- net S7P1: now also U1.65 (PC8)
- net S7P2: now also U1.66 (PC9)
- net S7P3: now also U1.78 (PC10)
- net S7P4: now also U1.79 (PC11)
- net S8P1: now also U1.80 (PC12)
- net S8P2: now also U1.7 (PC13)
- net S8P3: now also U1.8 (PC14)
- net S8P4: now also U1.9 (PC15)
- net S9P1: now also U1.55 (PD8)
- net S9P2: now also U1.56 (PD9)
- net S9P3: now also U1.57 (PD10)
- net S9P4: now also U1.58 (PD11)
- net SCK: now also J23.9 (Pin_9)
- net SCL: now also J23.7 (Pin_7)
- net SDA: now also J23.8 (Pin_8)
- net TX: now also J23.1 (Pin_1)
- new net: U15.13 (GND), U15.17 (GND)
Other:
- moved on the sheet: ADDR1
